Commit message: Add second joint and base to urdf

File: urdf/arm.urdf (robot description, URDF)
Before this commit: robot my_arm, 2 links, 1 joints
Links:
- removed link my_new_link
- added link base_column_link; visual cylinder length=0.5 radius=0.05
- added link extending_link; visual cylinder length=0.5 radius=0.05
Joints:
- removed joint my_joint
- added joint base_yaw_joint: type revolute, parent base_link, child base_column_link, origin xyz=0 0 0.025 rpy=0 0 0, axis 0 0 1, limit lower=-3 upper=3 effort=30 velocity=1.0
- added joint extending_joint: type revolute, parent base_column_link, child extending_link, origin xyz=0 0 0.5 rpy=0 1.57 0, axis 0 1 0, limit lower=-3 upper=3 effort=30 velocity=1.0

Commit message: Slightly change the urdf arm code (limits and renaming), mostly research today

File: urdf/arm.urdf (robot description, URDF)
Before this commit: robot my_arm, 3 links, 2 joints
Links:
- removed link extending_link
- added link horizontal_arm_base_link; visual cylinder length=0.5 radius=0.05
- link base_column_link: geometry 
- link base_link: geometry 
Joints:
- removed joint extending_joint
- added joint arm_pitch_joint: type revolute, parent base_column_link, child horizontal_arm_base_link, origin xyz=0 0 0.5 rpy=0 1.57 0, axis 0 1 0, limit lower=-1 upper=1 effort=30 velocity=1.0
- joint base_yaw_joint: limit lower=-3 upper=3 effort=30 velocity=1.0 -> lower=-3.6 upper=3.6 effort=30 velocity=1.0
